Commit message: applied recent ros1 changes

File: urdf/mini2_description.urdf (robot description, URDF)
Before this commit: robot mini2_description, 20 links, 19 joints
Links:
- added link 10_Link, mass 0.0625; collision mesh filename=package://mini2_description/meshes/lffoot.STL; visual mesh filename=package://mini2_description/meshes/lffoot.STL
- added link 20_Link, mass 0.0625; collision mesh filename=package://mini2_description/meshes/rffoot.STL; visual mesh filename=package://mini2_description/meshes/rffoot.STL
- added link 30_Link, mass 0.0625; collision mesh filename=package://mini_pupper_description/meshes/rbfoot.STL; visual mesh filename=package://mini_pupper_description/meshes/rbfoot.STL
- added link 40_Link, mass 0.0625; collision mesh filename=package://mini2_description/meshes/lbfoot.STL; visual mesh filename=package://mini2_description/meshes/lbfoot.STL
- added link lidar_link, mass 0.27; collision mesh filename=package://mini2_description/meshes/lidar.STL; visual mesh filename=package://mini2_description/meshes/lidar.STL
- added link odom
Joints:
- removed joint world_fixed
- added joint 10_Joint: type fixed, parent 11_Link, child 10_Link, origin xyz=0.001 -0.0759880541805861 0 rpy=-1.57079632679488 0 0, axis 0 0 0
- added joint 20_Joint: type fixed, parent 21_Link, child 20_Link, origin xyz=0.001 -0.0759880541805861 0 rpy=-1.57079632679488 0 0, axis 0 0 0
- added joint 30_Joint: type fixed, parent 31_Link, child 30_Link, origin xyz=0.001 -0.0759880541805861 0 rpy=-1.57079632679488 0 0, axis 0 0 0
- added joint 40_Joint: type fixed, parent 41_Link, child 40_Link, origin xyz=0.001 -0.0759880541805861 0 rpy=-1.57079632679488 0 0, axis 0 0 0
- added joint lidar_joint: type fixed, parent base_link, child lidar_link, origin xyz=-0.070475 0.0001 0.055 rpy=0 0 -1.5708, axis 0 0 0
- added joint odom_to_base_link: type fixed, parent odom, child base_link
- added joint world_to_odom: type fixed, parent world, child odom, origin xyz=0 0 0.1 rpy=0 0 0
