Commit message: revised launch params; added initial configs for champ

File: urdf/mini2_description_base.urdf (robot description, URDF)
Before this commit: robot mini2_description, 25 links, 24 joints
Links:
- added link odom
Joints:
- removed joint base_fixed
- added joint base_to_odom: type fixed, parent base_footprint, child odom, origin xyz=0 0 0.1 rpy=0 0 0
- added joint odom_to_base_link: type fixed, parent odom, child base_link
- joint 11_Joint: axis 0 0 1 -> 0 0  1
- joint 12_Joint: axis 0 0 1 -> 0 0  1
- joint 13_Joint: axis 0 0 1 -> 0 0  1
